File: PCB/Smart Smoker PCB.kicad_sch (KiCad schematic)
At the start: 1 part

Commit message: Added ESP32 board pcb files
Parts:
- removed U?: ESP32-WROOM-32, RF_Module:ESP32-WROOM-32, symbol RF_Module:ESP32-WROOM-32
- added U1: ESP32-WROOM-32UE_16MB, Customs Smoker:ESP32-WROOM-32UE 16MB, symbol ESP32-WROOM-32UE:ESP32-WROOM-32UE_16MB
Changed lines of the file:
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@@
 (kicad_sch (version 20211123) (generator eeschema)
   (paper "A4")
-  (symbol (lib_id "RF_Module:ESP32-WROOM-32") (at 135.89 101.6 0) (unit 1)
+  (symbol (lib_id "ESP32-WROOM-32UE:ESP32-WROOM-32UE_16MB") (at 100.33 63.5 0) (unit 1)
     (in_bom yes) (on_board yes) (fields_autoplaced)
-    (property "Reference" "U?" (id 0) (at 137.9094 63.5 0)
-      (effects (font (size 1.27 1.27)) (justify left))
+    (property "Reference" "U1" (id 0) (at 140.97 49.53 0)
+      (effects (font (size 1.524 1.524)))
     )
-    (property "Value" "ESP32-WROOM-32" (id 1) (at 137.9094 66.04 0)
-      (effects (font (size 1.27 1.27)) (justify left))
+    (property "Value" "ESP32-WROOM-32UE_16MB" (id 1) (at 140.97 53.34 0)
+      (effects (font (size 1.524 1.524)))
     )
-    (property "Footprint" "RF_Module:ESP32-WROOM-32" (id 2) (at 135.89 139.7 0)
+    (property "Footprint" "Customs Smoker:ESP32-WROOM-32UE 16MB" (id 2) (at 140.97 54.864 0)
+      (effects (font (size 1.524 1.524)) hide)
+    )
+    (property "Datasheet" "" (id 3) (at 100.33 63.5 0)
+      (effects (font (size 1.524 1.524)) hide)
+    )
+    (property "Manufacturer" "Espressif Systems" (id 4) (at 100.33 63.5 0)
       (effects (font (size 1.27 1.27)) hide)
     )
-    (property "Datasheet" "https://www.espressif.com/sites/default/files/documentation/esp32-wroom-32_datasheet_en.pdf" (id 3) (at 128.27 100.33 0)
+    (property "Manufacturer Part Number" "ESP32-WROOM-32UE-N8" (id 5) (at 100.33 63.5 0)
+      (effects (font (size 1.27 1.27)) hide)
+    )
+    (property "Vendor" "Digikey" (id 6) (at 100.33 63.5 0)
+      (effects (font (size 1.27 1.27)) hide)
+    )
+    (property "Vendor Part Number" "1965-ESP32-WROOM-32UE-N8CT-ND" (id 7) (at 100.33 63.5 0)
       (effects (font (size 1.27 1.27)) hide)
     )
@@
     (pin "39")
     (pin "4")
+    (pin "40")
+    (pin "41")
+    (pin "42")
+    (pin "43")
+    (pin "44")
+    (pin "45")
+    (pin "46")
+    (pin "47")
     (pin "5")
     (pin "6")
@@
   )
   (symbol_instances
-    (path "/4a6f9f76-50d6-4ae4-86e0-fc7dc15a31cd"
-      (reference "U?") (unit 1) (value "ESP32-WROOM-32") (footprint "RF_Module:ESP32-WROOM-32")
+    (path "/80a7e135-8f94-43f8-93fb-5e5903019107"
+      (reference "U1") (unit 1) (value "ESP32-WROOM-32UE_16MB") (footprint "Customs Smoker:ESP32-WROOM-32UE 16MB")
     )
   )

Commit message: Significant PCB progress
Parts:
- removed U1: ESP32-WROOM-32UE_16MB, Customs Smoker:ESP32-WROOM-32UE 16MB, symbol ESP32-WROOM-32UE:ESP32-WROOM-32UE_16MB
- added C1: 22uF 450V 20%, Capacitor_THT:CP_Radial_D16.0mm_P7.50mm, symbol Device:C
- added C2: 1000pF 440VAC Y5P, Capacitor_THT:C_Disc_D9.0mm_W5.0mm_P7.50mm, symbol Device:C
- added C3: 820uF 20% 16V, Capacitor_THT:CP_Radial_D10.0mm_P5.00mm, symbol Device:C
- added C4: 150uF 20% 35V, Capacitor_THT:CP_Radial_D8.0mm_P3.50mm, symbol Device:C
- added C5, C6: 0.1uF 50V X7R 0603, Capacitor_SMD:C_0603_1608Metric, symbol Device:C
- added D1: TVS DIODE 7VWM 12VC SMB, Diode_SMD:D_SMB, symbol Device:D_TVS
- added D2: LED, LED_SMD:LED_0603_1608Metric, symbol Device:LED
- added F1: 300V 1A SlowBlow, Fuse:Fuse_Littelfuse_395Series, symbol Device:Fuse
- added J1: AC_IN, Connector_Molex:Molex_Micro-Fit_3.0_43045-0400_2x02_P3.00mm_Horizontal, symbol Connector_Generic:Conn_02x02_Top_Bottom
- added J2: Hopper, Connector_Molex:Molex_Micro-Fit_3.0_43045-0400_2x02_P3.00mm_Horizontal, symbol Connector_Generic:Conn_02x02_Top_Bottom
- added J3: Lid, Connector_Molex:Molex_Micro-Fit_3.0_43045-0400_2x02_P3.00mm_Horizontal, symbol Connector_Generic:Conn_02x02_Top_Bottom
- added J?: Screw_Terminal_01x02, symbol Connector:Screw_Terminal_01x02
- added L1: 2.2mH 350mA 3.2Ohm TH, Inductor_THT:L_Radial_D12.0mm_P5.00mm_Fastron_11P, symbol pspice:INDUCTOR
- added L2: 2.2uH 7.2A 11.5mOhm, Inductor_SMD:L_Taiyo-Yuden_NR-80xx, symbol pspice:INDUCTOR
- added PS1: LS10-13B03R3, CONV_LS10-13B03R3, symbol LS10-13B03R3:LS10-13B03R3
- added R1: 6.8Ohm 3W 5% 2512, Resistor_SMD:R_2512_6332Metric, symbol Device:R
- added R2: R_US, Resistor_SMD:R_0603_1608Metric, symbol Device:R_US
- added TP1, TP2: TestPoint_2Pole, TestPoint:TestPoint_2Pads_Pitch5.08mm_Drill1.3mm, symbol Connector:TestPoint_2Pole
- added U1: ESP32-WROOM-32UE_16MB, IC38_ESP32-WROOM-32UE 16MB_EXP, symbol 2023-02-16_02-57-43:ESP32-WROOM-32UE_16MB
- added U2: DG409LEDY-T1-GE3, SOIC16_NARROW_VIS, symbol dg409:DG409LEDY-T1-GE3
- added U3: MAX31855KASA, Package_SO:SOIC-8_3.9x4.9mm_P1.27mm, symbol Sensor_Temperature:MAX31855KASA
Connections:
- new net: L1.2, PS1.2 (AC(L))
- new net: C1.1, PS1.3 (+V(CAP))
- new net: C1.2, C2.1, PS1.4 (-V(CAP))
- new net: C3.1, L2.1, PS1.6 (+VO)
- new net: F1.2, R1.1
- new net: L1.1, R1.2
- new net: D2.2 (A), R2.2
- new net +3.3V: C4.1, C5.1, C6.1, D1.2 (A2), J2.4 (Pin_4), J3.4 (Pin_4), L2.2, R2.1, TP2.1, U3.4 (VCC)
- new net AC_L: F1.1, J1.1 (Pin_1), TP1.1
- new net AC_N: J1.2 (Pin_2), PS1.1 (AC(N)), TP1.2
- new net GND: C2.2, C3.2, C4.2, C5.2, C6.2, D1.1 (A1), D2.1 (K), J2.2 (Pin_2), J3.2 (Pin_2), PS1.5 (-VO), TP2.2, U3.1 (GND)
- new net SCL: J2.3 (Pin_3), J3.3 (Pin_3)
- new net SDA: J2.1 (Pin_1), J3.1 (Pin_1)

Commit message: PCB layout done
Parts:
- removed J1: AC_IN, Connector_Molex:Molex_Micro-Fit_3.0_43045-0400_2x02_P3.00mm_Horizontal, symbol Connector_Generic:Conn_02x02_Top_Bottom
- removed J?: Screw_Terminal_01x02, symbol Connector:Screw_Terminal_01x02
- added C10, C15: 1uF 25V X5R 0603, Capacitor_SMD:C_0603_1608Metric, symbol Device:C
- added C11, C12, C13, C14, C3, C5: 0.1uF 50V X7R 0603, Capacitor_SMD:C_0603_1608Metric, symbol Device:C
- added C2: 22uF 10V X5R 0805, Capacitor_SMD:C_0805_2012Metric, symbol Device:C
- added C4: 0.01uF 50V X7R 0603, Capacitor_SMD:C_0603_1608Metric, symbol Device:C
- added C6: 4.7uF 25V X5R 0805, Capacitor_SMD:C_0805_2012Metric, symbol Device:C
- added C7, C8, C9: 10uF 16V X5R 0805, Capacitor_SMD:C_0805_2012Metric, symbol Device:C
- added D1: SP0503BAHT, Package_TO_SOT_SMD:SOT-143, symbol Power_Protection:SP0503BAHT
- added D3: Y 2V 20mA, LED_SMD:LED_0603_1608Metric, symbol Device:LED
- added D4: Y/G 2.2V 20mA, LED_SMD:LED_0603_1608Metric, symbol Device:LED
- added H1, H2, H3, H4: MountingHole, MountingHole:MountingHole_3.2mm_M3_DIN965_Pad, symbol Mechanical:MountingHole
- added J1: 105017-0001, MOLEX_105017-0001, symbol 105017-0001:105017-0001
- added J2, J3, J4, J5, J6: 393570002, CONN_393570002_MOL, symbol 0393570002:393570002
- added JP1: Jumper_2_Open, Connector_PinHeader_2.54mm:PinHeader_1x02_P2.54mm_Vertical, symbol Jumper:Jumper_2_Open
- added Q1, Q4: Q_PMOS_GSD, Customs Smoker:VESM_TOS, symbol Device:Q_PMOS_GSD
- added Q2, Q3: 25V 1.5A Trans, Package_TO_SOT_SMD:SOT-23-3, symbol Transistor_BJT:S8050
- added Q5, Q6: 2N7002T-7-F, Package_TO_SOT_SMD:SOT-23, symbol Transistor_FET:2N7002
- added R1, R12, R2, R3: 1kOhm 1% 0603, Resistor_SMD:R_0603_1608Metric, symbol Device:R_US
- added R10: 47.5kOhm 1% 0603, Resistor_SMD:R_0603_1608Metric, symbol Device:R_US
- added R11: 470Ohm 5% 0603, Resistor_SMD:R_0603_1608Metric, symbol Device:R_US
- added R13, R14, R4, R6, R7: 10K 1% 0603, Resistor_SMD:R_0603_1608Metric, symbol Device:R_US
- added R16: 470Ohm 1% 0603, Resistor_SMD:R_0603_1608Metric, symbol Device:R_US
- added R17: 140Ohm 1% 0603, Resistor_SMD:R_0603_1608Metric, symbol Device:R_US
- added R5: 22.1kOhm 1% 0603, Resistor_SMD:R_0603_1608Metric, symbol Device:R_US
- added R8, R9: 0Ohm 0603, Resistor_SMD:R_0603_1608Metric, symbol Device:R_US
- added S? (x2): TL1015AF160QG, Customs Smoker:SW_TL1015AF160QG, symbol TL1015AF160QG:TL1015AF160QG
- added U4: AMS1117-3.3, Package_TO_SOT_SMD:SOT-223-3_TabPin2, symbol Regulator_Linear:AMS1117-3.3
- added U5: CP2102N-Axx-xQFN28, Package_DFN_QFN:QFN-28-1EP_5x5mm_P0.5mm_EP3.35x3.35mm, symbol Interface_USB:CP2102N-Axx-xQFN28
- added U6: LTC4412xS6, Package_TO_SOT_SMD:TSOT-23-6, symbol Power_Management:LTC4412xS6
- C16: renamed from C1; footprint Capacitor_THT:CP_Radial_D16.0mm_P7.50mm -> Capacitor_THT:CP_Radial_D12.5mm_P5.00mm; Manufacturer Part Number UCS2W220MHD -> UCY2W220MHD; Vendor Part Number 493-5884-ND -> 493-6894-ND
- D5: renamed from D2; value LED -> R 1.8V 2mA 0603; Manufacturer (none) -> Rohm Semiconductor; Manufacturer Part Number (none) -> CSL1901UW1; Vendor (none) -> Digikey; Vendor Part Number (none) -> 846-CSL1901UW1CT-ND
- F1: value 300V 1A SlowBlow -> 300V 2A SlowBlow; Manufacturer Part Number 36911000000 -> 36912000000; Vendor Part Number F5459CT-ND -> F5461CT-ND
- R18: renamed from R2; value R_US -> 750Ohm 1% 0603; Manufacturer (none) -> YAGEO; Manufacturer Part Number (none) -> RC0603FR-07750RL; Vendor (none) -> Digikey; Vendor Part Number (none) -> 311-750HRCT-ND
- U1: footprint IC38_ESP32-WROOM-32UE 16MB_EXP -> Customs Smoker:ESP32-WROOM-32UE 16MB; Manufacturer (none) -> Espressif Systems; Manufacturer Part Number (none) -> ESP32-WROOM-32UE-N4; Vendor (none) -> Digikey; Vendor Part Number (none) -> 1965-ESP32-WROOM-32UE-N4CT-ND
- renumbered C6 to C1, C3 to C17, C4 to C18, C5 to C19, C2 to C20, D1 to D2, J2 to J7, J3 to J8, R1 to R15
Connections:
- net SCL is gone; now on net I2C_SCL: J7.3 (Pin_3), J8.3 (Pin_3)
- net SDA is gone; now on net I2C_SDA: J7.1 (Pin_1), J8.1 (Pin_1)
- net +3.3V: now also U1.2 (3V3), U2.14 (V+), U2.2 (EN), C10.2, C2.2, C3.2, C5.2, C6.2, JP1.1 (A), Q1.2 (S), Q4.2 (S), R1.2, R11.2, R14.2, R16.1, R2.2, R3.2, U5.6 (VDD), U5.7 (VREGIN), U6.6 (SENSE); no longer C18.1, C19.1, D2.2 (A2), L2.2
- net AC_L: now also J3.1
- net AC_N: now also J3.2
- net GND: now also U1.1 (GND), U1.15 (GND), U1.38 (GND), U1.39 (GND), U1.40 (GND), U1.41 (GND), U1.42 (GND), U1.43 (GND), U1.44 (GND), U1.45 (GND), U1.46 (GND), U1.47 (GND), U2.15 (GND), U2.3 (V-), C10.1, C11.2, C12.2, C13.1, C14.1, C15.2, C2.1, C3.1, C5.1, C6.1, C7.2, C8.2, C9.2, D1.1 (A), D4.1 (K), J1.5 (GND), Q5.2 (S), Q6.2 (S), R10.1, R13.2, R7.1, S?.1, S?.1, U4.1 (GND), U5.29 (GND), U5.3 (GND), U6.2 (GND), U6.3 (CTL)
- net MUX_OUT_-: now reaches U3.2 (T-)
- net MUX_OUT_-: now also U2.8 (DA), C4.2
- net MUX_OUT_+: now reaches U3.3 (T+)
- net MUX_OUT_+: now also U2.9 (DB), C4.1
- net SPI_SCK: now reaches U3.5 (SCK)
- net SPI_SCK: now also U1.30 (IO18)
- net SPI_CS: now reaches U3.6 (~{CS})
- net SPI_CS: now also U1.29 (IO5)
- net SPI_MISO: now reaches U3.7 (SO)
- net SPI_MISO: now also U1.31 (IO19)
- net IO2: now reaches U2.1 (A0)
- net IO2: now also U1.24 (IO2)
- net Probe4+: now reaches U2.10 (S4B)
- net Probe4+: now also J2.1
- net Probe3+: now reaches U2.11 (S3B)
- net Probe3+: now also J6.1
- net Probe2+: now reaches U2.12 (S2B)
- net Probe2+: now also J5.1
- net Probe1+: now reaches U2.13 (S1B)
- net Probe1+: now also J4.1
- net IO15: now reaches U2.16 (A1)
- net IO15: now also U1.23 (IO15)
- net Probe1-: now reaches U2.4 (S1A)
- net Probe1-: now also J4.2
- net Probe2-: now reaches U2.5 (S2A)
- net Probe2-: now also J5.2
- net Probe3-: now reaches U2.6 (S3A)
- net Probe3-: now also J6.2
- net Probe4-: now reaches U2.7 (S4A)
- net Probe4-: now also J2.2
- net IO25: now reaches U1.10 (IO25)
- net IO26: now reaches U1.11 (IO26)
- net IO27: now reaches U1.12 (IO27)
- net IO14: now reaches U1.13 (IO14)
- net IO12: now reaches U1.14 (IO12)
- net IO13: now reaches U1.16 (IO13)
- net IO0: now reaches U1.25 (IO0)
- net IO0: now also C14.2, Q3.3 (C), S?.2
- net IO4: now reaches U1.26 (IO4)
- net IO4: now also Q1.1 (G), R11.1, U6.4 (STAT)
- net IO16: now reaches U1.27 (IO16)
- net IO17: now reaches U1.28 (IO17)
- net IO17: now also D3.1 (K)
- net EN: now reaches U1.3 (EN)
- net EN: now also C15.1, Q2.3 (C), R14.1, S?.2
- net I2C_SDA: now reaches U1.33 (IO21)
- net I2C_SDA: now also R2.1
- net RXD0: now reaches U1.34 (RXD0)
- net RXD0: now also R9.1
- net TXD0: now reaches U1.35 (TXD0)
- net TXD0: now also R8.1
- net I2C_SCL: now reaches U1.36 (IO22)
- net I2C_SCL: now also R1.1
- net IO23: now reaches U1.37 (IO23)
- net IO23: now also R12.1
- net I36: now reaches U1.4 (SENSOR_VP)
- net I39: now reaches U1.5 (SENSOR_VN)
- net I34: now reaches U1.6 (IO34)
- net I35: now reaches U1.7 (IO35)
- net IO32: now reaches U1.8 (IO32)
- net IO33: now reaches U1.9 (IO33)
- new net: C13.2, JP1.2 (B), Q5.1 (G), Q6.1 (G), R12.2, R13.1
- new net: D3.2 (A), R16.2
- new net: Q4.1 (G), U6.5 (GATE)
- new net: R10.2, R5.2, U5.8 (VBUS)
- new net: R3.1, U5.9 (~{RST})
- new net: R7.2, U5.11 (~{SUSPEND})
- new net: D4.2 (A), R17.2
- new net: Q2.2 (B), R4.2
- new net: Q3.2 (B), R6.2
- new net +3.3VA: C12.1, C18.1, C19.1, D2.2 (A2), L2.2, Q4.3 (D), U6.1 (VIN)
- new net +3.3VP: C8.1, C9.1, Q1.3 (D), U4.2 (VO)
- new net +5V: C11.1, C7.1, D1.4 (K), J1.1 (VDD), R17.1, R5.1, U4.3 (VI)
- new net CTS: U5.23 (~{CTS})
- new net DTR: Q3.1 (E), R4.1, U5.28 (~{DTR})
- new net RTS: Q2.1 (E), R6.1, U5.24 (~{RTS})
- new net RXD: R8.2, U5.25 (RXD)
- new net TXD: R9.2, U5.26 (TXD)
- new net USB_DN: D1.3 (K), J1.2 (D-), Q6.3 (D), U5.4 (D+)
- new net USB_DP: D1.2 (K), J1.3 (D+), Q5.3 (D), U5.5 (D-)
- no-connect marks 0 -> 22
Other:
- note added: "AC/DC"
- note added: "Boot"
- note added: "Connectors"
- note added: "ESP32 MAIN"
- note added: "LEDs"
- note added: "NC by Default"
- note added: "Powerpath"
- note added: "Reset"
- note added: "Test Points"
- note added: "Thermocouples and Multiplexer"
- note added: "USB and Circuitry"
- moved on the sheet: C1, C16, C17, C18, C19, C20, D2, D5, F1, J7, J8, L1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

Commit message: Main PCB ready for review
Parts:
- gave numbers to parts that had none: 2

Commit message: Main pcb reviewed
Parts:
- added J2: 393570002, CONN_393570002_MOL, symbol 0393570002:393570002
- added JP2: Jumper_3_Open, Jumper:SolderJumper-3_P1.3mm_Open_RoundedPad1.0x1.5mm, symbol Jumper:Jumper_3_Open
- renumbered J2 to J3, J3 to J4, J4 to J5, J5 to J6, J6 to J7, J7 to J8, J8 to J9
Connections:
- net GND: now also JP2.2 (C)
- new net AC_G: J2.2, JP2.1 (A)
- new net TRG_GND: J2.1, JP2.3 (B)
