File: PCB/Smart Smoker PCB.kicad_sch (KiCad schematic)
At the start: 80 parts, among them J1 105017-0001, J2 393570002, J3 393570002, J4 393570002, J5 393570002, J6 393570002, J7 393570002, J8 Hopper, J9 Lid, Q1 Q_PMOS_GSD, Q2 25V 1.5A Trans, Q3 25V 1.5A Trans, Q4 Q_PMOS_GSD, Q5 2N7002T-7-F, Q6 2N7002T-7-F, U1 ESP32-WROOM-32UE_16MB, U2 DG409LEDY-T1-GE3, U3 MAX31855KASA, U4 AMS1117-3.3, U5 CP2102N-Axx-xQFN28, U6 LTC4412xS6

Commit message: Test on custom pcb initial
Parts:
- U4: footprint Package_TO_SOT_SMD:SOT-223-3_TabPin2 -> Package_TO_SOT_SMD:TO-252-3_TabPin2
Changed lines of the file:
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@@
     (property "Reference" "U4" (id 0) (at 306.07 110.49 0))
     (property "Value" "AMS1117-3.3" (id 1) (at 306.07 113.03 0))
-    (property "Footprint" "Package_TO_SOT_SMD:SOT-223-3_TabPin2" (id 2) (at 306.07 113.03 0)
+    (property "Footprint" "Package_TO_SOT_SMD:TO-252-3_TabPin2" (id 2) (at 306.07 113.03 0)
       (effects (font (size 1.27 1.27)) hide)
     )
@@
     )
     (path "/d4cc36e0-597d-4b97-98a3-66d07cb9fb5e"
-      (reference "U4") (unit 1) (value "AMS1117-3.3") (footprint "Package_TO_SOT_SMD:SOT-223-3_TabPin2")
+      (reference "U4") (unit 1) (value "AMS1117-3.3") (footprint "Package_TO_SOT_SMD:TO-252-3_TabPin2")
     )
     (path "/4ebcb3a9-02b7-497d-b880-0baa7dffd1dc"
