File: PCB/LID PCB/LIDPCB.kicad_pcb (KiCad board)
At the start: 2 copper layers, 22 x 17 mm, 10 parts, among them J1 POWER/I2C, U1 LTR-329ALS-01, U2 LSM6DSMTR

Commit message: 3x PCB ordered
Routing:
- net GND: track 6.63 -> 6.09 mm
Changed lines of the file:
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@@
   (segment (start 119.275 108) (end 119.275 109.731198) (width 0.65) (layer "F.Cu") (net 1))
   (segment (start 102.75 108.825) (end 103.825 108.825) (width 0.65) (layer "F.Cu") (net 1))
-  (segment (start 119 113.215) (end 119 113.34) (width 0.25) (layer "F.Cu") (net 1))
   (segment (start 120.075 112.79) (end 119.425 112.79) (width 0.25) (layer "F.Cu") (net 1))
   (segment (start 119.66 115) (end 119.66 115.64) (width 0.25) (layer "F.Cu") (net 1))
@@
   (segment (start 119.425 112.79) (end 119 113.215) (width 0.25) (layer "F.Cu") (net 1))
   (segment (start 117.185 115.785) (end 118 115.785) (width 0.25) (layer "F.Cu") (net 1))
-  (segment (start 115.525 113.5) (end 115.5 113.475) (width 0.25) (layer "F.Cu") (net 1))
   (segment (start 110.75 112) (end 112.05 112) (width 0.65) (layer "F.Cu") (net 1))
   (segment (start 120.3 113.015) (end 120.075 112.79) (width 0.25) (layer "F.Cu") (net 1))
@@
   (segment (start 118 115.785) (end 118 115.16) (width 0.25) (layer "F.Cu") (net 1))
   (segment (start 115.5 113.475) (end 113.525 113.475) (width 0.65) (layer "F.Cu") (net 1))
-  (segment (start 113.525 113.475) (end 113.5 113.45) (width 0.65) (layer "F.Cu") (net 1))
   (segment (start 116.5 113.5) (end 115.525 113.5) (width 0.25) (layer "F.Cu") (net 1))
   (segment (start 105.3 110.3) (end 109.05 110.3) (width 0.65) (layer "F.Cu") (net 1))
@@
   (segment (start 119.515 115.785) (end 119.815 115.785) (width 0.25) (layer "F.Cu") (net 1))
   (segment (start 117.34 113.5) (end 116.5 113.5) (width 0.25) (layer "F.Cu") (net 1))
-  (segment (start 115.5 114.7) (end 115.9 114.3) (width 0.25) (layer "F.Cu") (net 2))
-  (segment (start 115.5 115.025) (end 115.5 114.7) (width 0.25) (layer "F.Cu") (net 2))
   (segment (start 118.74 114.54) (end 118.5 114.3) (width 0.25) (layer "F.Cu") (net 2))
   (segment (start 118.5 114.3) (end 117.4 114.3) (width 0.25) (layer "F.Cu") (net 2))
@@
   (segment (start 117.34 114.24) (end 117.34 114) (width 0.25) (layer "F.Cu") (net 2))
   (segment (start 117.4 114.3) (end 117.34 114.24) (width 0.25) (layer "F.Cu") (net 2))
-  (via (at 116.2 109.4) (size 0.5) (drill 0.25) (layers "F.Cu" "B.Cu") (free) (net 2))
-  (via (at 113.6 105.2) (size 0.5) (drill 0.25) (layers "F.Cu" "B.Cu") (free) (net 2))
-  (via (at 118.5 114.3) (size 0.5) (drill 0.25) (layers "F.Cu" "B.Cu") (free) (net 2))
-  (via (at 120.7 106.9) (size 0.5) (drill 0.25) (layers "F.Cu" "B.Cu") (free) (net 2))
-  (via (at 109.1 115) (size 0.5) (drill 0.25) (layers "F.Cu" "B.Cu") (free) (net 2))
-  (via (at 101.3 105.7) (size 0.5) (drill 0.25) (layers "F.Cu" "B.Cu") (free) (net 2))
-  (via (at 120.7 109.6) (size 0.5) (drill 0.25) (layers "F.Cu" "B.Cu") (free) (net 2))
-  (via (at 115.9 114.3) (size 0.5) (drill 0.25) (layers "F.Cu" "B.Cu") (free) (net 2))
-  (via (at 114.7 112) (size 0.5) (drill 0.25) (layers "F.Cu" "B.Cu") (free) (net 2))
-  (via (at 109.5 101.4) (size 0.5) (drill 0.25) (layers "F.Cu" "B.Cu") (free) (net 2))
-  (segment (start 115.9 114.3) (end 118.5 114.3) (width 0.25) (layer "B.Cu") (net 2))
+  (via (at 116.2 109.4) (size 0.5) (drill 0.3) (layers "F.Cu" "B.Cu") (free) (net 2))
+  (via (at 113.6 105.2) (size 0.5) (drill 0.3) (layers "F.Cu" "B.Cu") (free) (net 2))
+  (via (at 118.5 114.3) (size 0.5) (drill 0.3) (layers "F.Cu" "B.Cu") (free) (net 2))
+  (via (at 120.7 106.9) (size 0.5) (drill 0.3) (layers "F.Cu" "B.Cu") (free) (net 2))
+  (via (at 109.1 115) (size 0.5) (drill 0.3) (layers "F.Cu" "B.Cu") (free) (net 2))
+  (via (at 101.3 105.7) (size 0.5) (drill 0.3) (layers "F.Cu" "B.Cu") (free) (net 2))
+  (via (at 120.7 109.6) (size 0.5) (drill 0.3) (layers "F.Cu" "B.Cu") (free) (net 2))
+  (via (at 116.3 116.1) (size 0.5) (drill 0.3) (layers "F.Cu" "B.Cu") (free) (net 2))
+  (via (at 114.7 112) (size 0.5) (drill 0.3) (layers "F.Cu" "B.Cu") (free) (net 2))
+  (via (at 109.5 101.4) (size 0.5) (drill 0.3) (layers "F.Cu" "B.Cu") (free) (net 2))
+  (segment (start 116.3 116.1) (end 118.1 114.3) (width 0.25) (layer "B.Cu") (net 2))
+  (segment (start 118.1 114.3) (end 118.5 114.3) (width 0.25) (layer "B.Cu") (net 2))
   (segment (start 102.75 107.175) (end 102.75 104.2875) (width 0.25) (layer "F.Cu") (net 3))
   (segment (start 118 113.34) (end 118 112.8) (width 0.16) (layer "F.Cu") (net 4))
   (segment (start 117.1 111.1) (end 117.9 111.1) (width 0.16) (layer "F.Cu") (net 4))
   (segment (start 117.462476 111.9) (end 117.7 111.9) (width 0.16) (layer "F.Cu") (net 4))
-  (segment (start 117.9 111.1) (end 118 111) (width 0.16) (layer "F.Cu") (net 4))
   (segment (start 118 111.6) (end 118 111.55) (width 0.16) (layer "F.Cu") (net 4))
   (segment (start 117.7 112.5) (end 117.462476 112.5) (width 0.16) (layer "F.Cu") (net 4))
   (segment (start 118 111.55) (end 118 111) (width 0.16) (layer "F.Cu") (net 4))
-  (via (at 117.1 111.1) (size 0.5) (drill 0.25) (layers "F.Cu" "B.Cu") (net 4))
+  (via (at 117.1 111.1) (size 0.5) (drill 0.3) (layers "F.Cu" "B.Cu") (net 4))
   (arc (start 117.162476 112.2) (mid 117.250344 111.987868) (end 117.462476 111.9) (width 0.16) (layer "F.Cu") (net 4))
   (arc (start 117.462476 112.5) (mid 117.250344 112.412132) (end 117.162476 112.2) (width 0.16) (layer "F.Cu") (net 4))
@@
   (segment (start 118.7302 111) (end 119.199998 111) (width 0.16) (layer "F.Cu") (net 5))
   (segment (start 118.6302 111.1) (end 118.7302 111) (width 0.16) (layer "F.Cu") (net 5))
-  (segment (start 119.299998 111.1) (end 119.199998 111) (width 0.16) (layer "F.Cu") (net 5))
   (segment (start 118.6302 111.2302) (end 118.6302 111.1) (width 0.16) (layer "F.Cu") (net 5))
   (segment (start 119.18515 111.87525) (end 119.18515 111.8302) (width 0.16) (layer "F.Cu") (net 5))
@@
   (segment (start 120 111.1) (end 119.299998 111.1) (width 0.16) (layer "F.Cu") (net 5))
   (segment (start 118.5 113.34) (end 118.5 112.9) (width 0.16) (layer "F.Cu") (net 5))
-  (via (at 120 111.1) (size 0.5) (drill 0.25) (layers "F.Cu" "B.Cu") (net 5))
+  (via (at 120 111.1) (size 0.5) (drill 0.3) (layers "F.Cu" "B.Cu") (net 5))
   (arc (start 118.907675 112.152725) (mid 119.103879 112.071454) (end 119.18515 111.87525) (width 0.16) (layer "F.Cu") (net 5))
   (arc (start 118.6302 112.4302) (mid 118.711471 112.233996) (end 118.907675 112.152725) (width 0.16) (layer "F.Cu") (net 5))
