File: PCB/LightSensorPCB/LightSensorPCB.kicad_sch (KiCad schematic)
At the start: 1 part, among them J1 POWER/I2C

Commit message: Light detection PCB
Parts:
- added C?: C, symbol Device:C
- added R? (x2): R_US, symbol Device:R_US
- added U?: LTR-329ALS-01, LTR-329ALS-01_LTO, symbol LTR-329-ALS:LTR-329ALS-01
Connections:
- net +3.3V: now also C?.1, U?.1 (VDD)
- net GND: now also C?.2, U?.2 (GND)
Changed lines of the file:
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@@
 (kicad_sch (version 20211123) (generator eeschema)
   (paper "A4")
+  (junction (at 140.97 73.66) (diameter 0) (color 0 0 0 0)
+  )
+  (junction (at 140.97 58.42) (diameter 0) (color 0 0 0 0)
+  )
+  (wire (pts (xy 140.97 68.58) (xy 140.97 73.66))
+    (stroke (width 0) (type default) (color 0 0 0 0))
+  )
   (wire (pts (xy 100.33 35.56) (xy 106.68 35.56))
     (stroke (width 0) (type default) (color 0 0 0 0))
   )
+  (wire (pts (xy 140.97 58.42) (xy 161.29 58.42))
+    (stroke (width 0) (type default) (color 0 0 0 0))
+  )
   (wire (pts (xy 76.2 35.56) (xy 87.63 35.56))
+    (stroke (width 0) (type default) (color 0 0 0 0))
+  )
+  (wire (pts (xy 161.29 60.96) (xy 161.29 73.66))
+    (stroke (width 0) (type default) (color 0 0 0 0))
+  )
+  (wire (pts (xy 140.97 73.66) (xy 161.29 73.66))
+    (stroke (width 0) (type default) (color 0 0 0 0))
+  )
+  (wire (pts (xy 140.97 58.42) (xy 140.97 60.96))
+    (stroke (width 0) (type default) (color 0 0 0 0))
+  )
+  (wire (pts (xy 140.97 48.26) (xy 140.97 58.42))
     (stroke (width 0) (type default) (color 0 0 0 0))
   )
@@
   (label "SCL" (at 106.68 35.56 180)
     (effects (font (size 1.27 1.27)) (justify right bottom))
+  )
+  (symbol (lib_id "Device:C") (at 140.97 64.77 0) (unit 1)
+    (in_bom yes) (on_board yes) (fields_autoplaced)
+    (property "Reference" "C?" (id 0) (at 144.78 63.4999 0)
+      (effects (font (size 1.27 1.27)) (justify left))
+    )
+    (property "Value" "C" (id 1) (at 144.78 66.0399 0)
+      (effects (font (size 1.27 1.27)) (justify left))
+    )
+    (property "Footprint" "" (id 2) (at 141.9352 68.58 0)
+      (effects (font (size 1.27 1.27)) hide)
+    )
+    (property "Datasheet" "~" (id 3) (at 140.97 64.77 0)
+      (effects (font (size 1.27 1.27)) hide)
+    )
+    (pin "1")
+    (pin "2")
+  )
+  (symbol (lib_id "power:GND") (at 140.97 73.66 0) (unit 1)
+    (in_bom yes) (on_board yes) (fields_autoplaced)
+    (property "Reference" "#PWR?" (id 0) (at 140.97 80.01 0)
+      (effects (font (size 1.27 1.27)) hide)
+    )
+    (property "Value" "GND" (id 1) (at 140.97 78.74 0))
+    (property "Footprint" "" (id 2) (at 140.97 73.66 0)
+      (effects (font (size 1.27 1.27)) hide)
+    )
+    (property "Datasheet" "" (id 3) (at 140.97 73.66 0)
+      (effects (font (size 1.27 1.27)) hide)
+    )
+    (pin "1")
+  )
+  (symbol (lib_id "LTR-329-ALS:LTR-329ALS-01") (at 161.29 58.42 0) (unit 1)
+    (in_bom yes) (on_board yes) (fields_autoplaced)
+    (property "Reference" "U?" (id 0) (at 181.61 46.99 0)
+      (effects (font (size 1.524 1.524)))
+    )
+    (property "Value" "LTR-329ALS-01" (id 1) (at 181.61 50.8 0)
+      (effects (font (size 1.524 1.524)))
+    )
+    (property "Footprint" "LTR-329ALS-01_LTO" (id 2) (at 181.61 52.324 0)
+      (effects (font (size 1.524 1.524)) hide)
+    )
+    (property "Datasheet" "" (id 3) (at 161.29 58.42 0)
+      (effects (font (size 1.524 1.524)))
+    )
+    (pin "1")
+    (pin "2")
+    (pin "3")
+    (pin "4")
+  )
+  (symbol (lib_id "Device:R_US") (at 209.55 54.61 90) (unit 1)
+    (in_bom yes) (on_board yes) (fields_autoplaced)
+    (property "Reference" "R?" (id 0) (at 209.55 48.26 90))
+    (property "Value" "R_US" (id 1) (at 209.55 50.8 90))
+    (property "Footprint" "" (id 2) (at 209.804 53.594 90)
+      (effects (font (size 1.27 1.27)) hide)
+    )
+    (property "Datasheet" "~" (id 3) (at 209.55 54.61 0)
+      (effects (font (size 1.27 1.27)) hide)
+    )
+    (pin "1")
+    (pin "2")
+  )
+  (symbol (lib_id "power:+3.3V") (at 140.97 48.26 0) (unit 1)
+    (in_bom yes) (on_board yes) (fields_autoplaced)
+    (property "Reference" "#PWR?" (id 0) (at 140.97 52.07 0)
+      (effects (font (size 1.27 1.27)) hide)
+    )
+    (property "Value" "+3.3V" (id 1) (at 140.97 43.18 0))
+    (property "Footprint" "" (id 2) (at 140.97 48.26 0)
+      (effects (font (size 1.27 1.27)) hide)
+    )
+    (property "Datasheet" "" (id 3) (at 140.97 48.26 0)
+      (effects (font (size 1.27 1.27)) hide)
+    )
+    (pin "1")
   )
   (symbol (lib_id "power:GND") (at 76.2 35.56 0) (unit 1)
@@
     (pin "4")
   )
+  (symbol (lib_id "Device:R_US") (at 209.55 44.45 90) (unit 1)
+    (in_bom yes) (on_board yes) (fields_autoplaced)
+    (property "Reference" "R?" (id 0) (at 209.55 38.1 90))
+    (property "Value" "R_US" (id 1) (at 209.55 40.64 90))
+    (property "Footprint" "" (id 2) (at 209.804 43.434 90)
+      (effects (font (size 1.27 1.27)) hide)
+    )
+    (property "Datasheet" "~" (id 3) (at 209.55 44.45 0)
+      (effects (font (size 1.27 1.27)) hide)
+    )
+    (pin "1")
+    (pin "2")
+  )
   (sheet_instances
     (path "/" (page "1"))
@@
       (reference "#PWR0102") (unit 1) (value "GND") (footprint "")
     )
+    (path "/1ecb137d-76d7-4e19-b42f-2d7da942d1c1"
+      (reference "#PWR?") (unit 1) (value "GND") (footprint "")
+    )
+    (path "/85d2645d-cc1c-443b-a073-4f80ce1df99c"
+      (reference "#PWR?") (unit 1) (value "+3.3V") (footprint "")
+    )
+    (path "/1ca43b8b-d13d-4f65-be5f-2c264b7e2696"
+      (reference "C?") (unit 1) (value "C") (footprint "")
+    )
     (path "/8c54ecc5-ac6f-4d45-94e0-d80a1a50bace"
       (reference "J1") (unit 1) (value "POWER/I2C") (footprint "Connector_Molex:Molex_Micro-Fit_3.0_43045-0412_2x02_P3.00mm_Vertical")
     )
-  )
+    (path "/5cee3aee-678c-4979-82ff-f2c3529676df"
+      (reference "R?") (unit 1) (value "R_US") (footprint "")
+    )
+    (path "/c0d5557b-f069-48dd-915d-6f7b515c3c4e"
+      (reference "R?") (unit 1) (value "R_US") (footprint "")
+    )
+    (path "/48b5e7aa-74d1-4daf-939c-91e123232bde"
+      (reference "U?") (unit 1) (value "LTR-329ALS-01") (footprint "LTR-329ALS-01_LTO")
+    )
+  )

Commit message: Light detection PCB
Parts:
- removed R?: R_US, symbol Device:R_US
- added D?: RED 1.8V 2mA, LED_SMD:LED_0603_1608Metric, symbol Device:LED
- added R2: 10kOhm 1% 0402, Resistor_SMD:R_0402_1005Metric, symbol Device:R_US
- added R?: 750Ohm 1% 0402, Resistor_SMD:R_0402_1005Metric, symbol Device:R_US
- C1: renamed from C?; value C -> 1 uF 6.3V X7R 0402; footprint (none) -> Capacitor_SMD:C_0402_1005Metric; Manufacturer (none) -> Murata Electronics; Manufacturer Part Number (none) -> GRM155R70J105KA12J; Vendor (none) -> Digikey; Vendor Part Number (none) -> 490-13339-1-ND
- R1: renamed from R?; value R_US -> 10kOhm 1% 0402; footprint (none) -> Resistor_SMD:R_0402_1005Metric; Manufacturer (none) -> YAGEO; Manufacturer Part Number (none) -> AC0402FR-0710KL; Vendor (none) -> Digikey; Vendor Part Number (none) -> YAG3436CT-ND
- U1: renamed from U?; footprint LTR-329ALS-01_LTO -> Customs:LTR-329ALS-01; Manufacturer (none) -> Lite-On Inc.; Manufacturer Part Number (none) -> LTR-329ALS-01; Vendor (none) -> Digikey; Vendor Part Number (none) -> 160-2160-1-ND
Connections:
- net +3.3V: now also R1.2, R2.2, R?.2
- net GND: now also D?.1 (K)
- net SCL: now also R1.1, U1.4 (SCL)
- net SDA: now also U1.3 (SDA), R2.1
- new net: D?.2 (A), R?.1
Other:
- moved on the sheet: R1

Commit message: Light detection PCB finished
Parts:
- added H1, H2: M3, MountingHole:MountingHole_3.2mm_M3_DIN965_Pad, symbol Mechanical:MountingHole
- J1: footprint Connector_Molex:Molex_Micro-Fit_3.0_43045-0412_2x02_P3.00mm_Vertical -> Connector_JST:JST_GH_SM04B-GHS-TB_1x04-1MP_P1.25mm_Horizontal; Manufacturer Molex -> JST; Manufacturer Part Number 0430450413 -> SM04B-GHS-TB(LF)(SN); Vendor Part Number WM2649-ND -> 455-1566-1-ND
- gave numbers to parts that had none: 2
Changed lines of the file:
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@@
     (pin "1")
+  )
+  (symbol (lib_id "Mechanical:MountingHole") (at 209.55 95.25 0) (unit 1)
+    (in_bom yes) (on_board yes) (fields_autoplaced)
+    (property "Reference" "H2" (id 0) (at 212.09 93.9799 0)
+      (effects (font (size 1.27 1.27)) (justify left))
+    )
+    (property "Value" "M3" (id 1) (at 212.09 96.5199 0)
+      (effects (font (size 1.27 1.27)) (justify left))
+    )
+    (property "Footprint" "MountingHole:MountingHole_3.2mm_M3_DIN965_Pad" (id 2) (at 209.55 95.25 0)
+      (effects (font (size 1.27 1.27)) hide)
+    )
+    (property "Datasheet" "~" (id 3) (at 209.55 95.25 0)
+      (effects (font (size 1.27 1.27)) hide)
+    )
   )
   (symbol (lib_id "Device:LED") (at 52.07 78.74 180) (unit 1)
     (in_bom yes) (on_board yes) (fields_autoplaced)
-    (property "Reference" "D?" (id 0) (at 53.6575 71.12 0))
+    (property "Reference" "D1" (id 0) (at 53.6575 71.12 0))
     (property "Value" "RED 1.8V 2mA" (id 1) (at 53.6575 73.66 0))
     (property "Footprint" "LED_SMD:LED_0603_1608Metric" (id 2) (at 52.07 78.74 0)
@@
   (symbol (lib_id "power:+3.3V") (at 19.05 74.93 0) (unit 1)
     (in_bom yes) (on_board yes) (fields_autoplaced)
-    (property "Reference" "#PWR?" (id 0) (at 19.05 78.74 0)
+    (property "Reference" "#PWR0106" (id 0) (at 19.05 78.74 0)
       (effects (font (size 1.27 1.27)) hide)
     )
@@
     (property "Reference" "J1" (id 0) (at 93.98 26.67 0))
     (property "Value" "POWER/I2C" (id 1) (at 93.98 29.21 0))
-    (property "Footprint" "Connector_Molex:Molex_Micro-Fit_3.0_43045-0412_2x02_P3.00mm_Vertical" (id 2) (at 92.71 33.02 0)
+    (property "Footprint" "Connector_JST:JST_GH_SM04B-GHS-TB_1x04-1MP_P1.25mm_Horizontal" (id 2) (at 92.71 33.02 0)
       (effects (font (size 1.27 1.27)) hide)
     )
@@
       (effects (font (size 1.27 1.27)) hide)
     )
-    (property "Manufacturer" "Molex" (id 4) (at 92.71 33.02 0)
-      (effects (font (size 1.27 1.27)) hide)
-    )
-    (property "Manufacturer Part Number" "0430450413" (id 5) (at 92.71 33.02 0)
+    (property "Manufacturer" "JST" (id 4) (at 92.71 33.02 0)
+      (effects (font (size 1.27 1.27)) hide)
+    )
+    (property "Manufacturer Part Number" "SM04B-GHS-TB(LF)(SN)" (id 5) (at 92.71 33.02 0)
       (effects (font (size 1.27 1.27)) hide)
     )
@@
       (effects (font (size 1.27 1.27)) hide)
     )
-    (property "Vendor Part Number" "WM2649-ND" (id 7) (at 92.71 33.02 0)
+    (property "Vendor Part Number" "455-1566-1-ND" (id 7) (at 92.71 33.02 0)
       (effects (font (size 1.27 1.27)) hide)
     )
@@
   (symbol (lib_id "power:GND") (at 69.85 82.55 0) (unit 1)
     (in_bom yes) (on_board yes) (fields_autoplaced)
-    (property "Reference" "#PWR?" (id 0) (at 69.85 88.9 0)
+    (property "Reference" "#PWR0107" (id 0) (at 69.85 88.9 0)
       (effects (font (size 1.27 1.27)) hide)
     )
@@
   (symbol (lib_id "Device:R_US") (at 34.29 78.74 270) (unit 1)
     (in_bom yes) (on_board yes) (fields_autoplaced)
-    (property "Reference" "R?" (id 0) (at 34.29 72.39 90))
+    (property "Reference" "R3" (id 0) (at 34.29 72.39 90))
     (property "Value" "750Ohm 1% 0402" (id 1) (at 34.29 74.93 90))
     (property "Footprint" "Resistor_SMD:R_0402_1005Metric" (id 2) (at 34.036 79.756 90)
@@
     )
     (pin "1")
+  )
+  (symbol (lib_id "Mechanical:MountingHole") (at 200.66 95.25 0) (unit 1)
+    (in_bom yes) (on_board yes) (fields_autoplaced)
+    (property "Reference" "H1" (id 0) (at 203.2 93.9799 0)
+      (effects (font (size 1.27 1.27)) (justify left))
+    )
+    (property "Value" "M3" (id 1) (at 203.2 96.5199 0)
+      (effects (font (size 1.27 1.27)) (justify left))
+    )
+    (property "Footprint" "MountingHole:MountingHole_3.2mm_M3_DIN965_Pad" (id 2) (at 200.66 95.25 0)
+      (effects (font (size 1.27 1.27)) hide)
+    )
+    (property "Datasheet" "~" (id 3) (at 200.66 95.25 0)
+      (effects (font (size 1.27 1.27)) hide)
+    )
   )
   (sheet_instances
@@
     )
     (path "/8064ce56-be3e-4761-96c0-c52b6787a81a"
-      (reference "#PWR?") (unit 1) (value "+3.3V") (footprint "")
+      (reference "#PWR0106") (unit 1) (value "+3.3V") (footprint "")
     )
     (path "/96fbe11d-0cef-4d98-a690-d60ab7dd8c80"
-      (reference "#PWR?") (unit 1) (value "GND") (footprint "")
+      (reference "#PWR0107") (unit 1) (value "GND") (footprint "")
     )
     (path "/1ca43b8b-d13d-4f65-be5f-2c264b7e2696"
@@
     )
     (path "/43e46a28-4813-4803-ba43-19d6d18b9f3e"
-      (reference "D?") (unit 1) (value "RED 1.8V 2mA") (footprint "LED_SMD:LED_0603_1608Metric")
+      (reference "D1") (unit 1) (value "RED 1.8V 2mA") (footprint "LED_SMD:LED_0603_1608Metric")
+    )
+    (path "/fb3f1a0d-1baa-48f5-b97b-213365732fa8"
+      (reference "H1") (unit 1) (value "M3") (footprint "MountingHole:MountingHole_3.2mm_M3_DIN965_Pad")
+    )
+    (path "/20766cb6-edcb-48de-b664-adcbf39bb6af"
+      (reference "H2") (unit 1) (value "M3") (footprint "MountingHole:MountingHole_3.2mm_M3_DIN965_Pad")
     )
     (path "/8c54ecc5-ac6f-4d45-94e0-d80a1a50bace"
-      (reference "J1") (unit 1) (value "POWER/I2C") (footprint "Connector_Molex:Molex_Micro-Fit_3.0_43045-0412_2x02_P3.00mm_Vertical")
+      (reference "J1") (unit 1) (value "POWER/I2C") (footprint "Connector_JST:JST_GH_SM04B-GHS-TB_1x04-1MP_P1.25mm_Horizontal")
     )
     (path "/5cee3aee-678c-4979-82ff-f2c3529676df"
@@
     )
     (path "/db8c2358-4a05-463f-a843-2d0baabf1e2b"
-      (reference "R?") (unit 1) (value "750Ohm 1% 0402") (footprint "Resistor_SMD:R_0402_1005Metric")
+      (reference "R3") (unit 1) (value "750Ohm 1% 0402") (footprint "Resistor_SMD:R_0402_1005Metric")
     )
     (path "/48b5e7aa-74d1-4daf-939c-91e123232bde"

Commit message: Significant PCB progress
Parts:
- removed R1, R2: 10kOhm 1% 0402, Resistor_SMD:R_0402_1005Metric, symbol Device:R_US
- added C2, C3, C5: 0.1 uF 50V X7R 0603, Capacitor_SMD:C_0603_1608Metric, symbol Device:C
- added C4: 4.7 uF 6.3V X5R 0603, Capacitor_SMD:C_0603_1608Metric, symbol Device:C
- added R4: 10kOhm 1% 0603, Resistor_SMD:R_0603_1608Metric, symbol Device:R_US
- added TP1: TestPoint_2Pole, Connector_PinHeader_2.54mm:PinHeader_1x02_P2.54mm_Vertical, symbol Connector:TestPoint_2Pole
- added U2: LSM6DSMTR, Customs:PQFN50P300X250X86-14N, symbol LSM6DSMTR:LSM6DSMTR
- added U3: VL53L3CXV0DH/1, XDCR_VL53L3CXV0DH/1, symbol VL53L3CXV0DH_1:VL53L3CXV0DH/1
- C1: value 1 uF 6.3V X7R 0402 -> 1 uF 25V X5R 0603; footprint Capacitor_SMD:C_0402_1005Metric -> Capacitor_SMD:C_0603_1608Metric; Manufacturer Murata Electronics -> Samsung Electro-Mechanics; Manufacturer Part Number GRM155R70J105KA12J -> CL10A105KA8NNNC; Vendor Part Number 490-13339-1-ND -> 1276-1102-1-ND
- D1: value RED 1.8V 2mA -> RED 1.8V 2mA 0603; Manufacturer Vishay Semiconductor Opto Division -> Rohm Semiconductor; Manufacturer Part Number TLMS1000-GS08 -> CSL1901UW1; Vendor Part Number TLMS1000-GS08CT-ND -> 846-CSL1901UW1CT-ND
- J1: footprint Connector_JST:JST_GH_SM04B-GHS-TB_1x04-1MP_P1.25mm_Horizontal -> Connector_Molex:Molex_Micro-Fit_3.0_43045-0400_2x02_P3.00mm_Horizontal; Manufacturer JST -> Molex; Manufacturer Part Number SM04B-GHS-TB(LF)(SN) -> 0430450400; Vendor Part Number 455-1566-1-ND -> WM1814-ND
- R3: value 750Ohm 1% 0402 -> 750Ohm 1% 0603; footprint Resistor_SMD:R_0402_1005Metric -> Resistor_SMD:R_0603_1608Metric; Manufacturer Part Number RC0402FR-07750RL -> RC0603FR-07750RL; Vendor Part Number 311-750LRCT-ND -> 311-750HRCT-ND
Connections:
- net +3.3V: now also J1.4 (Pin_4), C2.2, C3.2, C4.1, C5.1, U2.12 (CS), U2.5 (VDDIO), U2.8 (VDD), U3.1 (AVDDVCSEL), U3.11 (AVDD); no longer J1.1 (Pin_1)
- net GND: now also C2.1, C3.1, C4.2, C5.2, R4.1, U2.1 (SDO/SA0), U2.2 (SDX), U2.3 (SCX), U2.6 (GND), U2.7 (GND), U3.12 (GND), U3.2 (AVSSVCSEL), U3.3 (GND), U3.4 (GND), U3.6 (GND)
- net SCL: now also J1.3 (Pin_3), U2.13 (SCL/SPC), U3.10 (SCL); no longer J1.4 (Pin_4)
- net SDA: now also J1.1 (Pin_1), U2.14 (SDA/SDI/SDO), U3.9 (SDA); no longer J1.3 (Pin_3)
- new net: R4.2, U3.5 (XSHUT)
- new net GPIO_LSM: TP1.1, U2.4 (INT1)
- new net GPIO_VL5: TP1.2, U3.7 (GPIO1)
- no-connect marks 0 -> 3
Other:
- note added: "CS pulled high for I2C"
- note added: "LSB i2c address 1101010b"
- note added: "VL5 i2c address 0x52 (1010010)"

Commit message: Main pcb reviewed
Changed lines of the file:
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@@
+    (stroke (width 0) (type default) (color 0 0 0 0))
+  )
+  (wire (pts (xy 201.93 60.96) (xy 209.55 60.96))
     (stroke (width 0) (type default) (color 0 0 0 0))
   )
@@
     (stroke (width 0) (type default) (color 0 0 0 0))
   )
-  (wire (pts (xy 201.93 58.42) (xy 267.97 58.42))
+  (wire (pts (xy 143.51 140.97) (xy 143.51 142.24))
     (stroke (width 0) (type default) (color 0 0 0 0))
   )
@@
     (stroke (width 0) (type default) (color 0 0 0 0))
   )
-  (wire (pts (xy 201.93 60.96) (xy 267.97 60.96))
-    (stroke (width 0) (type default) (color 0 0 0 0))
-  )
   (wire (pts (xy 111.76 35.56) (xy 100.33 35.56))
     (stroke (width 0) (type default) (color 0 0 0 0))
@@
     (stroke (width 0) (type default) (color 0 0 0 0))
   )
+  (wire (pts (xy 201.93 58.42) (xy 209.55 58.42))
+    (stroke (width 0) (type default) (color 0 0 0 0))
+  )
   (wire (pts (xy 124.46 107.95) (xy 124.46 104.14))
     (stroke (width 0) (type default) (color 0 0 0 0))
@@
     (stroke (width 0) (type default) (color 0 0 0 0))
   )
-  (wire (pts (xy 143.51 142.24) (xy 143.51 140.97))
-    (stroke (width 0) (type default) (color 0 0 0 0))
-  )
   (wire (pts (xy 205.74 130.81) (xy 215.9 130.81))
     (stroke (width 0) (type default) (color 0 0 0 0))
@@
     (effects (font (size 1.27 1.27)) (justify right bottom))
   )
-  (label "SCL" (at 267.97 58.42 180)
+  (label "SCL" (at 209.55 58.42 180)
     (effects (font (size 1.27 1.27)) (justify right bottom))
   )
@@
     (effects (font (size 1.27 1.27)) (justify left bottom))
   )
-  (label "SDA" (at 267.97 60.96 180)
-    (effects (font (size 1.27 1.27)) (justify right bottom))
-  )
+  (label "SDA" (at 209.55 60.96 180)
+    (effects (font (size 1.27 1.27)) (justify right bottom))
+  )
