File: PCB/Main PCB/REV B/_autosave-DigitalPCB.kicad_sch (KiCad schematic)
At the start: 107 parts, among them J1 DF12NC-20DS-0.5V_51_, J2 1050170001, J3 Hopper, J4 Screen, J5 Spare1, J6 Spare2, Q1 MBT3904DW1, U1 AMS1117-3.3, U2 ESP32-WROOM-32UE_16MB, U3 TPS2115APWR, U4 TLP2362TPR_E, U5 CP2102N-A02-GQFN24, U6 TLP2362TPR_E, U7 TLP2362TPR_E, U8 STM811SW16F

Commit message: PCB - digital routing first pass done
Parts:
- added C19: 0.1uF 50V X7R 0603, Capacitor_SMD:C_0603_1608Metric, symbol Device:C
- added C20: 0.01uF 50V X7R 0603, Capacitor_SMD:C_0603_1608Metric, symbol Device:C
- added U9: MAX31855KASA, Package_SO:SOIC-8_3.9x4.9mm_P1.27mm, symbol Sensor_Temperature:MAX31855KASA
Connections:
- net +3.3V: now also C19.1, U9.4 (VCC)
- net GND: now also C19.2, U9.1 (GND)
- net Probe1+: now also C20.1, U9.3 (T+)
- net Probe1-: now also C20.2, U9.2 (T-)
- net SPI_CS: now also U9.6 (~{CS})
- net SPI_MISO: now also U9.7 (SO)
- net SPI_SCK: now also U9.5 (SCK)
