File: PCB/Main PCB/REV B/DigitalPCB.kicad_sch (KiCad schematic)
At the start: 107 parts, among them J1 DF12NC-20DS-0.5V_51_, J2 1050170001, J3 Hopper, J4 Screen, J5 Spare1, J6 Spare2, Q1 MBT3904DW1, U1 AMS1117-3.3, U2 ESP32-WROOM-32UE_16MB, U3 TPS2115APWR, U4 TLP2362TPR_E, U5 CP2102N-A02-GQFN24, U6 TLP2362TPR_E, U7 TLP2362TPR_E, U8 STM811SW16F

Commit message: PCB - digital routing first pass done
Parts:
- added C?: 0.01uF 50V X7R 0603, Capacitor_SMD:C_0603_1608Metric, symbol Device:C
- added C?: 0.1uF 50V X7R 0603, Capacitor_SMD:C_0603_1608Metric, symbol Device:C
- added U?: MAX31855KASA, Package_SO:SOIC-8_3.9x4.9mm_P1.27mm, symbol Sensor_Temperature:MAX31855KASA
Connections:
- net +3.3V: now also C?.1, U?.4 (VCC)
- net GND: now also C?.2, U?.1 (GND)
- net Probe1+: now also C?.1, U?.3 (T+)
- net Probe1-: now also C?.2, U?.2 (T-)
- net SPI_CS: now also U?.6 (~{CS})
- net SPI_MISO: now also U?.7 (SO)
- net SPI_SCK: now also U?.5 (SCK)

Commit message: PCB - hopper pcb done routing ready for review
Parts:
- gave numbers to parts that had none: 3

Commit message: PCB - Text edited, all ready for review
Parts:
- added TP12, TP15, TP17: TP, TestPoint:TestPoint_Pad_D1.0mm, symbol Connector:TestPoint
- renumbered C19 to C11, C20 to C12, C11 to C13, C12 to C14, C13 to C15, C14 to C16, C15 to C17, C16 to C18, C17 to C19, C18 to C20, TP12 to TP13, TP13 to TP14, TP14 to TP16, TP15 to TP18, TP16 to TP19, TP17 to TP20, TP18 to TP21, TP19 to TP22, TP20 to TP23, TP21 to TP24, TP22 to TP25, TP23 to TP26, TP24 to TP27, U9 to U5, U5 to U6, U6 to U7, U7 to U8, U8 to U9
Connections:
- net Opto_Auger: now also TP12.1
- net Opto_Fan: now also TP15.1
- net Opto_Ignitor: now also TP17.1
