File: PCB/Main PCB/REV B/AnalogPCB.kicad_pcb (KiCad board)
At the start: 2 copper layers, 60 x 100 mm, 60 parts, among them J1 DF12NB_4.0_-20DP-0.5V_51_, J2 393570002, J3 393570002, J4 393570002, J5 393570002, J6 SJ3-35053D, Q1 2N7002, Q2 2N7002, Q3 2N7002, U1 ALDP105W, U2 ALDP105W, U3 ALDP105W

Commit message: Start rev C pcb, with analog first. Update passives to 0805
Parts:
- removed TP13, TP15, TP16, TP17, TP18, TP19, TP20, TP29: TP, TestPoint:TestPoint_Pad_D1.0mm
- added TP10: TP, TestPoint:TestPoint_Pad_D1.0mm, F.Cu at (175.5, 62.2)
- added TP11: TP, TestPoint:TestPoint_Pad_D1.0mm, F.Cu at (170.6, 66.0)
- added TP4: TP, TestPoint:TestPoint_Pad_D1.0mm, F.Cu at (181.1, 54.8)
- added TP5: TP, TestPoint:TestPoint_Pad_D1.0mm, F.Cu at (170.6, 69.0)
- added TP6: TP, TestPoint:TestPoint_Pad_D1.0mm, F.Cu at (133.2, 102.7)
- added TP7: TP, TestPoint:TestPoint_Pad_D1.0mm, F.Cu at (161.7, 75.8)
- added TP8: TP, TestPoint:TestPoint_Pad_D1.0mm, F.Cu at (128.8, 105.7)
- added TP9: TP, TestPoint:TestPoint_Pad_D1.0mm, F.Cu at (191.2, 48.8)
- C1, C3: value 0.1uF 50V X7R 0603 -> 0.1uF 50V X7R 0805; footprint Capacitor_SMD:C_0603_1608Metric -> Capacitor_SMD:C_0805_2012Metric; moved to F.Cu
- C2, C4, J6, JP4: moved to F.Cu
- D1, D7: value B 3.2 20mA 0603 -> B 3.2V 20mA 0805; footprint LED_SMD:LED_0603_1608Metric -> LED_SMD:LED_0805_2012Metric
- D2, D8: footprint Customs Smoker:RB521S30T1G-M -> Diode_SMD:D_SOD-323
- D3: value R 2.0V 20mA -> B 3.2V 20mA 0805; footprint LED_SMD:LED_0603_1608Metric -> LED_SMD:LED_0805_2012Metric
- D4: value R 2.0V 20mA -> Schottky 30v 200mA; footprint LED_SMD:LED_0603_1608Metric -> Diode_SMD:D_SOD-323
- D5: value B 3.2 20mA 0603 -> R 2.0V 20mA; footprint LED_SMD:LED_0603_1608Metric -> LED_SMD:LED_0805_2012Metric
- D6: value Schottky 30v 200mA -> R 2.0V 20mA; footprint Customs Smoker:RB521S30T1G-M -> LED_SMD:LED_0805_2012Metric
- J1: value DF12NB_4.0_-20DP-0.5V_51_ -> 393570002; footprint Customs Smoker:HRS_DF12NB_4.0_-20DP-0.5V_51_ -> Customs Smoker:CONN_393570002_MOL; moved to F.Cu
- J2: value 393570002 -> DF12NB_4.0_-20DP-0.5V_51_; footprint Customs Smoker:CONN_393570002_MOL -> Customs Smoker:HRS_DF12NB_4.0_-20DP-0.5V_51_
- R1, R9: value 91Ohm 1% 0603 -> 91Ohm 1% 0805; footprint Resistor_SMD:R_0603_1608Metric -> Resistor_SMD:R_0805_2012Metric
- R10, R2: value 10K 1% 0603 -> 10K 1% 0805; footprint Resistor_SMD:R_0603_1608Metric -> Resistor_SMD:R_0805_2012Metric
- R11, R3: value 0 Ohm 0603 -> 0 Ohm 0805; footprint Resistor_SMD:R_0603_1608Metric -> Resistor_SMD:R_0805_2012Metric
- R4: value 150Ohm 1% 0603 -> 91Ohm 1% 0805; footprint Resistor_SMD:R_0603_1608Metric -> Resistor_SMD:R_0805_2012Metric
- R5: value 64.9Ohm 1% 0603 -> 10K 1% 0805; footprint Resistor_SMD:R_0603_1608Metric -> Resistor_SMD:R_0805_2012Metric
- R6: value 91Ohm 1% 0603 -> 0 Ohm 0805; footprint Resistor_SMD:R_0603_1608Metric -> Resistor_SMD:R_0805_2012Metric
- R7: value 10K 1% 0603 -> 150Ohm 1% 0805; footprint Resistor_SMD:R_0603_1608Metric -> Resistor_SMD:R_0805_2012Metric
- R8: value 0 Ohm 0603 -> 64.9Ohm 1% 0805; footprint Resistor_SMD:R_0603_1608Metric -> Resistor_SMD:R_0805_2012Metric
- moved TC1 161.0 mm to (202.9, 78.8), turned to 0 degrees
- moved R13 153.4 mm to (177.4, 53.2)
- moved R12 146.2 mm to (171.7, 60.0)
- moved R10 145.9 mm to (187.4, 48.8), turned to 0 degrees
- moved R7 144.2 mm to (181.8, 51.8), turned to 0 degrees
- moved TP2 136.8 mm to (185.5, 51.8), turned to 0 degrees
- moved R3 136.4 mm to (183.0, 48.8), turned to 0 degrees
- moved R14 131.9 mm to (162.4, 66.9), turned to 0 degrees
- moved JP2 130.6 mm to (163.0, 49.1), turned to 0 degrees
- moved Q3 130.5 mm to (173.9, 49.5)
- moved JP4 130.3 mm to (163.0, 52.9), turned to 0 degrees
- moved J3 129.5 mm to (216.8, 82.7), turned to 0 degrees
- moved C1 128.2 mm to (178.6, 48.8), turned to 0 degrees
- moved JP1 125.1 mm to (168.7, 49.1), turned to 0 degrees
- moved R1 124.3 mm to (176.1, 56.2), turned to 0 degrees
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Connections:
- D3 pad 1: GND -> Net-(Q2-Pad3)
- D4 pad 1: GND -> +5V
- D4 pad 2: Net-(D4-Pad2) -> Net-(U2-Pad4)
- D5 pad 1: Net-(D5-Pad1) -> GND
- D6 pad 1: +5V -> GND
- D6 pad 2: Net-(D6-Pad2) -> Net-(R8-Pad2)
- J1 pad 1: +3.3VA -> /AC_L
- J1 pad 2: GND -> /AC_N
- J2 pad 1: /AC_L -> +3.3VA
- J2 pad 2: /AC_N -> GND
- Q2 pad 3: Net-(D5-Pad1) -> Net-(Q2-Pad3)
- R5 pad 1: +3.3VA -> Net-(JP2-Pad2)
- R5 pad 2: Net-(D4-Pad2) -> /Opto_Ignitor
- R6 pad 1: +5V -> Net-(U2-Pad4)
- R6 pad 2: Net-(D5-Pad2) -> Net-(Q2-Pad3)
- R7 pad 1: Net-(JP2-Pad2) -> +5V
- R7 pad 2: /Opto_Ignitor -> Net-(D5-Pad2)
- R8 pad 1: Net-(D6-Pad2) -> +3.3VA
- R8 pad 2: Net-(D5-Pad1) -> Net-(R8-Pad2)
- TP1 pad 1: +3.3VA -> /AC_N
- TP3 pad 1: +5V -> /AC_L
- U2 pad 4: Net-(D6-Pad2) -> Net-(U2-Pad4)
Routing:
- net +3.3VA: track 186.5 -> 0.00 mm, vias 15 -> 0
- net +5V: track 164.6 -> 0.00 mm, vias 13 -> 0
- net /AC_N: track 137.2 -> 0.00 mm
- net /MeatProbe+: track 137.1 -> 0.00 mm, vias 3 -> 0
- net /MeatProbe-: track 128.8 -> 0.00 mm, vias 3 -> 0
- net /AC_L: track 121.2 -> 0.00 mm
- net /Probe1-: track 102.7 -> 0.00 mm, vias 1 -> 0
- net /Opto_Fan: track 82.7 -> 0.00 mm, vias 3 -> 0
- net /Opto_Ignitor: track 81.0 -> 0.00 mm, vias 3 -> 0
- net /Probe1+: track 75.7 -> 0.00 mm, vias 3 -> 0
- net Net-(D6-Pad2): track 69.7 -> 0.00 mm, vias 1 -> 0
- net Net-(D2-Pad2): track 62.0 -> 0.00 mm, vias 1 -> 0
- net Net-(U3-Pad4): track 61.7 -> 0.00 mm, vias 1 -> 0
- net /Opto_Auger: track 57.0 -> 0.00 mm, vias 3 -> 0
- net Net-(D5-Pad1): track 48.4 -> 0.00 mm, vias 2 -> 0
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- removed copper zone on B.Cu, net GND
- removed copper zone on F.Cu, net GND
Other:
- outline, holes or cut-outs redrawn
- board text removed: "+3.3V"
- board text removed: "+5V"
- board text removed: "AC L"
- board text removed: "AC N"
- board text removed: "AUGER"
- board text removed: "DIMS: 100mm x 60mm HOLE: 10mm x 50mm"
- board text removed: "FAN"
- board text removed: "IGNITOR"
- board text removed: "IGNITR"
- board text removed: "SLEEVE"
- board text removed: "SMART SMOKER ANALOG - REV B MAY 2025"
- board text removed: "TIP"
