File: PCB/Main PCB/REV C/AnalogPCB.kicad_sch (KiCad schematic)
At the start: 60 parts, among them J1 DF12NB_4.0_-20DP-0.5V_51_, J2 393570002, J3 393570002, J4 393570002, J5 393570002, J6 SJ3-35053D, Q1 2N7002, Q2 2N7002, Q3 2N7002, U1 ALDP105W, U2 ALDP105W, U3 ALDP105W

Commit message: Start rev C pcb, with analog first. Update passives to 0805
Parts:
- removed C?: 0.1uF 50V X7R 0805, Capacitor_SMD:C_0805_2012Metric, symbol Device:C
- removed D? (x2): Schottky 30v 200mA, Diode_SMD:D_SOD-323, symbol Diode:1N6857UR
- removed D?: R 2.0V 20mA, LED_SMD:LED_0805_2012Metric, symbol Device:LED
- removed D? (x2): B 3.2V 20mA 0805, LED_SMD:LED_0805_2012Metric, symbol Device:LED
- removed R? (x2): 0 Ohm 0805, Resistor_SMD:R_0805_2012Metric, symbol Device:R_US
- removed R? (x2): 91Ohm 1% 0805, Resistor_SMD:R_0805_2012Metric, symbol Device:R_US
- removed R? (x2): 10K 1% 0805, Resistor_SMD:R_0805_2012Metric, symbol Device:R_US
- added C3: 0.1uF 50V X7R 0603, Capacitor_SMD:C_0603_1608Metric, symbol Device:C
- added D4: R 2.0V 20mA, LED_SMD:LED_0603_1608Metric, symbol Device:LED
- added D5, D7: B 3.2 20mA 0603, LED_SMD:LED_0603_1608Metric, symbol Device:LED
- added D6, D8: Schottky 30v 200mA, Customs Smoker:RB521S30T1G-M, symbol Diode:1N6857UR
- added R10, R7: 10K 1% 0603, Resistor_SMD:R_0603_1608Metric, symbol Device:R_US
- added R11, R8: 0 Ohm 0603, Resistor_SMD:R_0603_1608Metric, symbol Device:R_US
- added R6, R9: 91Ohm 1% 0603, Resistor_SMD:R_0603_1608Metric, symbol Device:R_US
- C1: value 0.1uF 50V X7R 0805 -> 0.1uF 50V X7R 0603; footprint Capacitor_SMD:C_0805_2012Metric -> Capacitor_SMD:C_0603_1608Metric; Manufacturer Part Number CL21B104KBCNNNC -> CL10B104KB8NNWC; Vendor Part Number 1276-1003-1-ND -> 1276-1935-1-ND
- D1: value B 3.2V 20mA 0805 -> B 3.2 20mA 0603; footprint LED_SMD:LED_0805_2012Metric -> LED_SMD:LED_0603_1608Metric; Manufacturer Part Number 150080BS75000 -> 150060BS75000; Vendor Part Number 732-4982-1-ND -> 732-4966-1-ND
- D2: footprint Diode_SMD:D_SOD-323 -> Customs Smoker:RB521S30T1G-M; Manufacturer Toshiba Semiconductor and Storage -> onsemi; Manufacturer Part Number CUS520,H3F -> RB521S30T1G; Vendor Part Number CUS520H3FCT-ND -> RB521S30T1GOSCT-ND
- D3: footprint LED_SMD:LED_0805_2012Metric -> LED_SMD:LED_0603_1608Metric; Manufacturer Part Number LS R976-NR-1-0-20-R18 -> LO Q976-PS-25-0-20-R18; Vendor Part Number 475-LSR976-NR-1CT-ND -> 475-LOQ976-PS-25-0-20-R18CT-ND
- R1: value 91Ohm 1% 0805 -> 91Ohm 1% 0603; footprint Resistor_SMD:R_0805_2012Metric -> Resistor_SMD:R_0603_1608Metric; Manufacturer Part Number AC0805FR-0791RL -> RC0603FR-0791RL; Vendor Part Number 13-AC0805FR-0791RLCT-ND -> 311-91.0HRCT-ND
- R2: value 10K 1% 0805 -> 10K 1% 0603; footprint Resistor_SMD:R_0805_2012Metric -> Resistor_SMD:R_0603_1608Metric; Manufacturer YAGEO -> Stackpole Electronics Inc; Manufacturer Part Number RC0805FR-0710KL -> RNCP0603FTD10K0; Vendor Part Number 311-10.0KCRCT-ND -> RNCP0603FTD10K0CT-ND
- R3: value 0 Ohm 0805 -> 0 Ohm 0603; footprint Resistor_SMD:R_0805_2012Metric -> Resistor_SMD:R_0603_1608Metric; Manufacturer Part Number RMCF0805ZT0R00 -> RC0603JR-070RL; Vendor Part Number RMCF0805ZT0R00CT-ND -> 311-0.0GRCT-ND
- R4: value 150Ohm 1% 0805 -> 150Ohm 1% 0603; footprint Resistor_SMD:R_0805_2012Metric -> Resistor_SMD:R_0603_1608Metric; Manufacturer Part Number RC0805FR-07150RL -> RC0603FR-07150RL; Vendor Part Number 311-150CRCT-ND -> 311-150HRCT-ND
- R5: value 64.9Ohm 1% 0805 -> 64.9Ohm 1% 0603; footprint Resistor_SMD:R_0805_2012Metric -> Resistor_SMD:R_0603_1608Metric; Manufacturer Part Number RC0805FR-0764R9L -> RC0603FR-0764R9L; Vendor Part Number 311-64.9CRCT-ND -> 311-64.9HRCT-ND
Connections:
- net +5V: now also C3.2, D6.1 (K), D8.1 (K), R6.1, R9.1
- net GND: now also C3.1, D4.1 (K)
- net Opto_Fan: now also R10.2
- net Opto_Ignitor: now also R7.2
- net at U3.4: now also D8.2 (A), R11.1
- net at Q3.3 (D): now also D7.1 (K), R11.2
- net at JP3.2 (C): now also R10.1
- net at R5.2, TP15.1: now also D4.2 (A)
- net at U2.4: now also D6.2 (A), R8.1
- net at JP2.2 (C): now also R7.1
- net at Q2.3 (D): now also D5.1 (K), R8.2
- new net: D7.2 (A), R9.2
- new net: D5.2 (A), R6.2
Other:
- note removed: "TODO Test this and fix"
