File: PCB/Main PCB/REV C/DigitalPCB.kicad_sch (KiCad schematic)
At the start: 109 parts, among them J1 DF12NC-20DS-0.5V_51_, J2 1050170001, J3 Hopper, J4 Screen, J5 Spare1, U1 AMS1117-3.3, U2 ESP32-WROOM-32UE_16MB, U3 TPS2115APWR, U4 TLP2362TPR_E, U5 MAX31855KASA, U6 CP2102N-A02-GQFN24, U7 TLP2362TPR_E, U8 TLP2362TPR_E

Commit message: begin change of power arch so mux occurs at 5.0v rather than 3.3v
Parts:
- removed C2: 22uF 16V X5R 0805, Capacitor_SMD:C_0805_2012Metric, symbol Device:C
- removed C?: 10uF 16V X5R 0805, Capacitor_SMD:C_0805_2012Metric, symbol Device:C
- removed D? (x2): R 2.0V 20mA, LED_SMD:LED_0805_2012Metric, symbol Device:LED
- removed R1, R?: 64.9Ohm 1% 0805, Resistor_SMD:R_0805_2012Metric, symbol Device:R_US
- removed U1: AMS1117-3.3, Package_TO_SOT_SMD:TO-252-2, symbol Regulator_Linear:AMS1117-3.3
- added C? (x3): 10uF 16V X5R 0805, Capacitor_SMD:C_0805_2012Metric, symbol Device:C
- added C?: 56uF 50V TH, Capacitor_THT:C_Radial_D10.0mm_H12.5mm_P5.00mm, symbol Device:C
- added D?: R 2.0V 20mA, LED_SMD:LED_0805_2012Metric, symbol Device:LED
- added L?: 5.6uH 2.9A, Customs Smoker:IND_IFSC-2020DE-01_VIS, symbol pspice:INDUCTOR
- added PS?: TSR-2-2433, Converter_DCDC:Converter_DCDC_TRACO_TSR-1_THT, symbol Regulator_Switching:TSR_1-2433
- added R?: 150Ohm 1% 0805, Resistor_SMD:R_0805_2012Metric, symbol Device:R_US
- added TP?: TP, TestPoint:TestPoint_Pad_D1.0mm, symbol Connector:TestPoint
Connections:
- net +3.3V: now also J1.1, J1.3, C?.1, C?.2, L?.2, TP?.1
- net +3.3VA: no longer J1.1, J1.3, J1.5, J1.7
- net +5V: now also PS?.1 (Vin), R?.1; no longer J1.11, J1.9, R?.1
- net +5VA: now also J1.11, J1.5, J1.7, J1.9; no longer C?.1, D6.4 (K), J2.1 (VBUS)
- net GND: now also C?.1, C?.1, C?.2, C?.2, D?.1 (K), PS?.2 (GND)
- new net: D?.2 (A), R?.2
- new net: C?.1, C?.2, L?.1, PS?.3 (Vout)
- new net +5VD: C?.1, D6.4 (K), J2.1 (VBUS), R?.1
Other:
- note added: "BUSES 5VA - ACDC 5VD - USB 5V - Main 3.3V - Main"
- note added: "change power arch to 5v from usb or converter then into ams once"
- note added: "todo - change out 0603 components - verify reset logic - verify usb chip - verify esp pinouts - confirm probe circuit - change connector - confirm loads - confirm power supplies X"
- note removed: "todo - change out 0603 components - verify reset logic - verify usb chip - verify esp pinouts - confirm probe circuit - change connector - confirm loads - confirm power supplies"
- moved on the sheet: D2, D?, R2, R?
